File: hardware/kicad/sam_cpu/sam_cpu.kicad_pcb (KiCad board)
At the start: 4 copper layers, 120.7 x 231.8 mm, 412 parts, among them J1 J1 SWITCH COLUMNS, J10 J10 SPEAKERS, J11 J11 POWER, J12 J12 SWITCH ROWS, J13 J13 DEDICATED, J17 EXT 5V, J18 J18 GI DIMMER, J19 USB-C (to Pi), J2 J2 DEDICATED, J20 SWD, J21 Raspberry Pi 40-pin, J3 J3 DEDICATED, J5 J5 DMD, J6 J6 SWITCH ROWS, J9 J9 IO BUS, Q1 AO3401A, Q11 MMBT3904, Q12 MMBT3904, Q13 MMBT3904, Q14 MMBT3904, Q15 MMBT3904, Q16 MMBT3904, Q17 MMBT3904, Q18 MMBT3904, Q2 AO3401A, Q3 2N7002, SW1 RESET, SW2 BOOTSEL, SW3 DIP x8, U1 LTC4412, U10 LM339, U11 LM339, U14 74HC165, U15 74HC165, U16 74HC165, U17 74HC165, U18 74HC165, U19 74HC165, U2 LTC4412, U20 74HC595, U21 74HCT245, U22 PCM5102A, U23 TDA2030A, U24 TDA2030A, U3 AMS1117-3.3, U4 RP2354B, U5 TPS3808G33, U6 SN74LVC8T245, U7 74AHCT541, U8 LM339, U9 LM339, Y1 12MHz

Commit message: PCB draft: keep only outline, holes and connectors on the board
Vincent will place and route the rest himself, so all other parts now
wait off the board, one block per schematic sheet.

Co-Authored-By: Claude Opus 5.5 (1M context) <noreply@anthropic.com>
Claude-Session: https://claude.ai/code/session_01ExuDVoDDDHhVWjb8EwVzYb
Parts:
- moved R62 282.4 mm to (327.7, 227.0)
- moved R63 282.4 mm to (331.3, 227.0)
- moved C30 280.6 mm to (324.3, 30.8)
- moved C32 280.6 mm to (331.6, 30.8)
- moved C31 280.6 mm to (328.0, 30.8)
- moved D13 276.4 mm to (323.4, 211.2)
- moved D14 276.4 mm to (328.8, 211.2)
- moved R89 268.9 mm to (221.7, 317.0)
- moved R90 268.9 mm to (225.3, 317.0)
- moved C46 268.3 mm to (324.1, 221.9)
- moved C47 268.3 mm to (327.8, 221.9)
- moved C43 268.3 mm to (313.2, 221.9)
- moved C45 268.3 mm to (320.5, 221.9)
- moved C44 268.3 mm to (316.8, 221.9)
- moved C48 268.3 mm to (331.4, 221.9)
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
Commit message: Add RTC, test points and stereo speaker connector; place all parts on 2 layers
Schematic: DS3231MZ real-time clock on the Pi I2C1 with a CR2032 holder,
22 test points (rails, bus, strobes, switch chain, VREF, DAC outputs) and
J22, a second KK-396 speaker connector with L and R as separate pairs.
ERC 0 errors, generated netlist matches the intended nets.

PCB: 2 copper layers. The RP2354B sits near J9 with its USB-C on the top
edge 13 mm from the USB pins; decoupling, regulator and crystal parts on
their pins; every other part grouped by sheet next to its connector, low
parts only under the Pi. J17 and J22 on the right edge; Pi and J5 12 mm
lower to fit the audio parts.

Co-Authored-By: Claude Opus 5.5 (1M context) <noreply@anthropic.com>
Claude-Session: https://claude.ai/code/session_01ExuDVoDDDHhVWjb8EwVzYb
Parts:
- added BT1: CR2032, Battery:BatteryHolder_Keystone_3034_1x20mm, F.Cu at (58.9, 145.0)
- added C119: 100n, Capacitor_SMD:C_0603_1608Metric, F.Cu at (72.0, 133.4)
- added J22: J22 STEREO, Connector_Molex:Molex_KK-396_A-41791-0004_1x04_P3.96mm_Vertical, F.Cu at (145.0, 60.0)
- added TP1: +5V, TestPoint:TestPoint_Pad_D1.5mm, F.Cu at (89.3, 103.5)
- added TP10: GND, TestPoint:TestPoint_Pad_D1.5mm, F.Cu at (83.7, 78.6)
- added TP11: J9_IOSTB, TestPoint:TestPoint_Pad_D1.5mm, F.Cu at (48.3, 82.2)
- added TP12: J9_NBRESET, TestPoint:TestPoint_Pad_D1.5mm, F.Cu at (51.5, 82.2)
- added TP13: J9_D0, TestPoint:TestPoint_Pad_D1.5mm, F.Cu at (54.7, 82.2)
- added TP14: J9_A0, TestPoint:TestPoint_Pad_D1.5mm, F.Cu at (57.9, 82.2)
- added TP15: STB1, TestPoint:TestPoint_Pad_D1.5mm, F.Cu at (119.8, 220.9)
- added TP16: STB2, TestPoint:TestPoint_Pad_D1.5mm, F.Cu at (123.0, 220.9)
- added TP17: SW_CLK, TestPoint:TestPoint_Pad_D1.5mm, F.Cu at (126.2, 220.9)
- added TP18: SW_DATA, TestPoint:TestPoint_Pad_D1.5mm, F.Cu at (129.4, 220.9)
- added TP19: VREF, TestPoint:TestPoint_Pad_D1.5mm, F.Cu at (48.3, 174.8)
- added TP2: +3V3, TestPoint:TestPoint_Pad_D1.5mm, F.Cu at (92.5, 103.5)
- added TP20: DAC_OUTL, TestPoint:TestPoint_Pad_D1.5mm, F.Cu at (130.7, 110.4)
- added TP21: DAC_OUTR, TestPoint:TestPoint_Pad_D1.5mm, F.Cu at (133.9, 110.4)
- added TP22: GND, TestPoint:TestPoint_Pad_D1.5mm, F.Cu at (137.1, 110.4)
- added TP3: +4V5, TestPoint:TestPoint_Pad_D1.5mm, F.Cu at (95.7, 103.5)
- added TP4: +12V, TestPoint:TestPoint_Pad_D1.5mm, F.Cu at (98.9, 103.5)
- added TP5: -12V, TestPoint:TestPoint_Pad_D1.5mm, F.Cu at (102.1, 103.5)
- added TP6: GND, TestPoint:TestPoint_Pad_D1.5mm, F.Cu at (105.3, 103.5)
- added TP7: GND, TestPoint:TestPoint_Pad_D1.5mm, F.Cu at (108.5, 103.5)
- added TP8: +1V1, TestPoint:TestPoint_Pad_D1.5mm, F.Cu at (65.3, 85.3)
- added TP9: RUN, TestPoint:TestPoint_Pad_D1.5mm, F.Cu at (68.5, 85.3)
- added U25: DS3231MZ, Package_SO:SOIC-8_3.9x4.9mm_P1.27mm, F.Cu at (77.4, 139.4)
- moved R61 278.7 mm to (48.5, 184.7)
- moved R62 278.7 mm to (52.2, 184.7)
- moved R63 278.7 mm to (55.8, 184.7)
- moved C30 277.6 mm to (47.5, 51.6), turned to 90 degrees
- moved C32 273.8 mm to (58.6, 51.8)
- moved C31 271.5 mm to (58.7, 65.0), turned to 90 degrees
- moved R90 267.3 mm to (48.5, 116.5)
- moved C65 266.7 mm to (48.2, 90.6), turned to 90 degrees
- moved D11 262.6 mm to (52.6, 174.7)
- moved D12 262.6 mm to (58.0, 174.7)
- moved D13 262.6 mm to (63.4, 174.7)
- moved D14 262.6 mm to (68.8, 174.7)
- moved C53 262.4 mm to (48.2, 158.6), turned to 90 degrees
- moved C33 261.3 mm to (61.4, 64.7), turned to 90 degrees
- moved Q3 260.0 mm to (60.3, 78.2)
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Connections:
- J21 pad 3: unconnected-(J21-SDA/GPIO2-Pad3) -> /MCU and Pi/PI_SDA
- J21 pad 5: unconnected-(J21-SCL/GPIO3-Pad5) -> /MCU and Pi/PI_SCL
Other:
- copper layers 4 -> 2

Commit message: Audio on external 12 V with TDA7297 stereo + subwoofer amps, NCP1117, guide regulator layout
- Remove the +-12 V input from J11; J23 external +12 V with polyfuse and TVS
- Replace the two TDA2030A with a TDA7297 bridge amp for left/right (J10, J22)
  and a second TDA7297 for the subwoofer (J24), fed by an (L+R)/2 110 Hz
  Sallen-Key low-pass (OPA1678); shared standby and RP2354B-controlled mute
- AMS1117 -> NCP1117-3.3 (ceramic-stable, as in the RP2350 guide), 10 uF 1206
- L1 and crystal part numbers from the RP2350 hardware guide
- Place the core regulator parts by hand following the Pico 2 layout; amps in a
  row with a heatsink keep-out; J23/J22/J24 on the right edge

Co-Authored-By: Claude Opus 5.5 (1M context) <noreply@anthropic.com>
Claude-Session: https://claude.ai/code/session_01ExuDVoDDDHhVWjb8EwVzYb
Parts:
- removed D27, D28, D29, D30: S1M, Diode_SMD:D_SMA
- removed FB2, FB3: 1A, Inductor_SMD:L_0805_2012Metric
- added C120: 10u, Capacitor_SMD:C_0805_2012Metric, F.Cu at (126.2, 110.1)
- added C121: 10u, Capacitor_SMD:C_0805_2012Metric, F.Cu at (130.3, 110.1)
- added D5: SMBJ15A, Diode_SMD:D_SMB, F.Cu at (109.6, 99.3)
- added F1: 4A hold, Fuse:Fuse_2920_7451Metric, F.Cu at (92.6, 100.0)
- added J23: EXT 12V, TerminalBlock_Phoenix:TerminalBlock_Phoenix_MKDS-1,5-2-5.08_1x02_P5.08mm_Horizontal, F.Cu at (144.5, 60.0)
- added J24: J24 SUBWOOFER, Connector_Molex:Molex_KK-396_A-41791-0004_1x04_P3.96mm_Vertical, F.Cu at (145.0, 89.5)
- added Q4: 2N7002, Package_TO_SOT_SMD:SOT-23, F.Cu at (127.2, 63.3)
- added R199: 22k, Resistor_SMD:R_0603_1608Metric, F.Cu at (133.8, 120.0)
- added R200: 1.8k, Resistor_SMD:R_0603_1608Metric, F.Cu at (137.4, 120.0)
- added R201: 10k, Resistor_SMD:R_0603_1608Metric, F.Cu at (115.5, 122.2)
- added R202: 10k, Resistor_SMD:R_0603_1608Metric, F.Cu at (119.2, 122.2)
- added R203: 100k, Resistor_SMD:R_0603_1608Metric, F.Cu at (122.8, 122.2)
- added U26: OPA1678, Package_SO:SOIC-8_3.9x4.9mm_P1.27mm, F.Cu at (132.7, 101.9)
- C105: value 22u -> 2.2n; footprint Capacitor_SMD:CP_Elec_6.3x7.7 -> Capacitor_SMD:C_0603_1608Metric
- C106: value 220n -> 1u
- C108, C118: value 100u -> 470u
- C109, C115: value 100n -> 1u
- C110, C116: value 100u -> 1u; footprint Capacitor_SMD:CP_Elec_6.3x7.7 -> Capacitor_SMD:C_0603_1608Metric
- C111: value 2.2n -> 100n
- C112: value 1u -> 220n
- C113: value 22u -> 100n; footprint Capacitor_SMD:CP_Elec_6.3x7.7 -> Capacitor_SMD:C_0603_1608Metric
- C114: value 220n -> 10u; footprint Capacitor_SMD:C_0603_1608Metric -> Capacitor_SMD:C_0805_2012Metric
- C2: value 47u -> 100u; footprint Capacitor_SMD:CP_Elec_6.3x7.7 -> Capacitor_SMD:CP_Elec_8x10
- C3: value 47u -> 100n; footprint Capacitor_SMD:CP_Elec_6.3x7.7 -> Capacitor_SMD:C_0603_1608Metric
- C6: footprint Capacitor_SMD:C_0805_2012Metric -> Capacitor_SMD:C_1206_3216Metric
- C7: value 22u -> 10u; footprint Capacitor_SMD:C_0805_2012Metric -> Capacitor_SMD:C_1206_3216Metric
- R189: value 4.7k -> 1.8k
- R190: value 22k -> 470
- R191: value 1k -> 22k
- R192: value 1 -> 1.8k; footprint Resistor_SMD:R_1206_3216Metric -> Resistor_SMD:R_0603_1608Metric
- R193: value 470 -> 20k
- R194: value 22k -> 20k
- R195: value 4.7k -> 100k
- R196: value 22k -> 10k
- R197: value 1k -> 10k
- R198: value 1 -> 10k; footprint Resistor_SMD:R_1206_3216Metric -> Resistor_SMD:R_0603_1608Metric
- TP10: value GND -> J9_IOSTB
- TP11: value J9_IOSTB -> J9_NBRESET
- TP12: value J9_NBRESET -> J9_D0
- TP13: value J9_D0 -> J9_A0
- TP14: value J9_A0 -> STB1
- TP15: value STB1 -> STB2
- TP16: value STB2 -> SW_CLK
- TP17: value SW_CLK -> SW_DATA
- TP18: value SW_DATA -> VREF
- TP19: value VREF -> DAC_OUTL
- TP20: value DAC_OUTL -> DAC_OUTR
- TP21: value DAC_OUTR -> SUB_OUT
- TP5: value -12V -> GND
- TP7: value GND -> +1V1
- TP8: value +1V1 -> RUN
- TP9: value RUN -> GND
- U23, U24: value TDA2030A -> TDA7297; footprint Package_TO_SOT_THT:TO-220-5_P3.4x3.7mm_StaggerOdd_Lead3.8mm_Vertical -> Package_TO_SOT_THT:TO-220-15_P2.54x5.08mm_StaggerOdd_Lead4.58mm_Vertical
- U3: value AMS1117-3.3 -> NCP1117-3.3
- moved TP14 151.9 mm to (119.8, 220.9)
- moved TP19 139.2 mm to (131.0, 62.9)
- moved TP18 93.3 mm to (48.3, 174.8)
- moved C8 60.5 mm to (51.7, 109.1)
- moved TP20 47.6 mm to (134.2, 62.9)
- moved C6 44.6 mm to (87.7, 56.8)
- moved C105 43.9 mm to (135.2, 113.1)
- moved C110 39.9 mm to (119.2, 115.7)
- moved U2 39.8 mm to (89.3, 64.9)
- moved TP10 35.6 mm to (48.3, 82.2)
- moved TP7 35.1 mm to (83.7, 78.6)
- moved C116 33.7 mm to (133.8, 115.7)
- moved C102 33.0 mm to (131.0, 66.3)
- moved C2 30.6 mm to (117.4, 51.4)
- moved C115 30.4 mm to (130.1, 115.7), turned to 0 degrees
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Connections:
- C103 pad 1: Net-(C103-Pad1) -> /Audio/AFL
- C104 pad 1: Net-(C103-Pad1) -> Net-(C104-Pad1)
- C104 pad 2: Net-(C104-Pad2) -> Net-(U23A-+)
- C105 pad 1: Net-(C105-Pad1) -> /Audio/AFR
- C106 pad 2: GND -> Net-(U23B-+)
- C109 pad 1: GND -> /Audio/AFL
- C109 pad 2: -12V -> Net-(C109-Pad2)
- C110 pad 1: GND -> /Audio/AFR
- C110 pad 2: -12V -> Net-(C110-Pad2)
- C111 pad 1: Net-(C111-Pad1) -> Net-(U26A-+)
- C112 pad 1: Net-(C111-Pad1) -> Net-(C112-Pad1)
- C112 pad 2: Net-(C112-Pad2) -> /Audio/SUB_OUT
- C113 pad 1: Net-(C113-Pad1) -> +12V
- C114 pad 1: Net-(C114-Pad1) -> Net-(U26B-+)
- C115 pad 1: +12V -> /Audio/SUB_OUT
- C115 pad 2: GND -> Net-(C115-Pad2)
- C116 pad 1: +12V -> Net-(C116-Pad1)
- C116 pad 2: GND -> Net-(U24A-+)
- C117 pad 1: GND -> +12V
- C117 pad 2: -12V -> GND
- C118 pad 1: GND -> +12V
- C118 pad 2: -12V -> GND
- C3 pad 1: GND -> +12V
- C3 pad 2: -12V -> GND
- J10 pad 1: Net-(D27-A) -> Net-(J10-Pin_1)
- J10 pad 2: Net-(D29-A) -> Net-(J10-Pin_2)
- J10 pad 3: GND -> Net-(J10-Pin_3)
- J10 pad 4: GND -> Net-(J10-Pin_4)
- J11 pad 3: Net-(J11-Pin_3) -> unconnected-(J11-Pin_3-Pad3)
- J11 pad 6: Net-(J11-Pin_6) -> unconnected-(J11-Pin_6-Pad6)
- J22 pad 1: Net-(D27-A) -> Net-(J10-Pin_1)
- J22 pad 2: GND -> Net-(J10-Pin_3)
- J22 pad 3: Net-(D29-A) -> Net-(J10-Pin_2)
- J22 pad 4: GND -> Net-(J10-Pin_4)
- R187 pad 2: Net-(C103-Pad1) -> /Audio/AFL
- R188 pad 1: Net-(C104-Pad2) -> /Audio/AFL
- R188 pad 2: Net-(U23-+) -> Net-(C104-Pad1)
- R189 pad 1: Net-(U23-+) -> Net-(C104-Pad1)
- R190 pad 1: Net-(U23--) -> Net-(U22-OUTR)
- R190 pad 2: Net-(D27-A) -> /Audio/AFR
- R191 pad 1: Net-(U23--) -> /Audio/AFR
- R191 pad 2: Net-(C105-Pad1) -> Net-(C106-Pad1)
- R192 pad 1: Net-(D27-A) -> Net-(C106-Pad1)
- R192 pad 2: Net-(C106-Pad1) -> GND
- R193 pad 1: Net-(U22-OUTR) -> Net-(C109-Pad2)
- R193 pad 2: Net-(C111-Pad1) -> Net-(C112-Pad1)
- R194 pad 1: Net-(C112-Pad2) -> Net-(C110-Pad2)
- R194 pad 2: Net-(U24-+) -> Net-(C112-Pad1)
- R195 pad 1: Net-(U24-+) -> Net-(C112-Pad1)
- R195 pad 2: GND -> Net-(U26B-+)
- R196 pad 1: Net-(U24--) -> Net-(C112-Pad1)
- R196 pad 2: Net-(D29-A) -> Net-(U26A-+)
- R197 pad 1: Net-(U24--) -> +12V
- R197 pad 2: Net-(C113-Pad1) -> Net-(U26B-+)
- R198 pad 1: Net-(D29-A) -> Net-(U26B-+)
- R198 pad 2: Net-(C114-Pad1) -> GND
- TP10 pad 1: GND -> Net-(J9-Pin_15)
- TP11 pad 1: Net-(J9-Pin_15) -> Net-(J9-Pin_13)
- TP12 pad 1: Net-(J9-Pin_13) -> Net-(J9-Pin_7)
- TP13 pad 1: Net-(J9-Pin_7) -> Net-(J9-Pin_12)
- TP14 pad 1: Net-(J9-Pin_12) -> Net-(J1-Pin_1)
- TP15 pad 1: Net-(J1-Pin_1) -> Net-(J1-Pin_3)
- TP16 pad 1: Net-(J1-Pin_3) -> SW_CLK
- TP17 pad 1: SW_CLK -> SW_DATA
- TP18 pad 1: SW_DATA -> VREF
- TP19 pad 1: VREF -> Net-(U22-OUTL)
- TP20 pad 1: Net-(U22-OUTL) -> Net-(U22-OUTR)
- TP21 pad 1: Net-(U22-OUTR) -> /Audio/SUB_OUT
- TP5 pad 1: -12V -> GND
- TP7 pad 1: GND -> +1V1
- TP8 pad 1: +1V1 -> Net-(U4-RUN)
- TP9 pad 1: Net-(U4-RUN) -> GND
- U23 pad 1: Net-(U23-+) -> Net-(J10-Pin_1)
- U23 pad 2: Net-(U23--) -> Net-(J10-Pin_3)
- U23 pad 3: -12V -> +12V
- U23 pad 4: Net-(D27-A) -> Net-(U23A-+)
- U23 pad 5: +12V -> unconnected-(U23A-NC-Pad5)
- U24 pad 1: Net-(U24-+) -> Net-(J24-Pin_1)
- U24 pad 2: Net-(U24--) -> Net-(J24-Pin_2)
- U24 pad 3: -12V -> +12V
- U24 pad 4: Net-(D29-A) -> Net-(U24A-+)
- U24 pad 5: +12V -> unconnected-(U24A-NC-Pad5)
- U4 pad 46: unconnected-(U4-GPIO37-Pad46) -> AMP_MUTE
Other:
- board text added: "HEATSINK FOR U23 / U24 (TDA7297): NO PARTS"

Commit message: Add two HD DMD panels on a PIO parallel bus (incremental edit)
RP2354B GPIO20-36 drive two HUB75 panels (J25/J26) through 3 x 74AHCT245
with shared CLK/LAT/OE and A/B row lines; J5 shares DMD_D0-D6. The 165
load and 595 latch share GPIO17; coin door moves to a 7th 165 (U30),
LED_STATUS and GI_SPARE to a new first 595 (U31). Board widened to 142 mm
below the Pi. Sheets and board edited in place via tools/changes, no
existing footprint moved.

Co-Authored-By: Claude Opus 5.5 (1M context) <noreply@anthropic.com>
Claude-Session: https://claude.ai/code/session_01ExuDVoDDDHhVWjb8EwVzYb
Parts:
- added C122: 100n, Capacitor_SMD:C_0603_1608Metric, F.Cu at (161.6, 215.5)
- added C123: 100n, Capacitor_SMD:C_0603_1608Metric, F.Cu at (161.6, 226.4)
- added C124: 100n, Capacitor_SMD:C_0603_1608Metric, F.Cu at (150.8, 237.3)
- added C125: 100n, Capacitor_SMD:C_0603_1608Metric, F.Cu at (144.7, 257.6)
- added C126: 100n, Capacitor_SMD:C_0603_1608Metric, F.Cu at (45.4, 197.4)
- added J25: J25 HUB75 PANEL A, Connector_IDC:IDC-Header_2x08_P2.54mm_Vertical, F.Cu at (154.6, 190.0)
- added J26: J26 HUB75 PANEL B, Connector_IDC:IDC-Header_2x08_P2.54mm_Vertical, F.Cu at (165.4, 190.0)
- added RN10: 33, Resistor_SMD:R_Array_Convex_4x0603, F.Cu at (164.1, 239.2)
- added RN11: 33, Resistor_SMD:R_Array_Convex_4x0603, F.Cu at (167.9, 239.2)
- added RN6: 33, Resistor_SMD:R_Array_Convex_4x0603, F.Cu at (152.5, 250.1)
- added RN7: 33, Resistor_SMD:R_Array_Convex_4x0603, F.Cu at (156.3, 250.1)
- added RN8: 33, Resistor_SMD:R_Array_Convex_4x0603, F.Cu at (160.1, 250.1)
- added RN9: 33, Resistor_SMD:R_Array_Convex_4x0603, F.Cu at (163.9, 250.1)
- added TP23: DMD_CLK, TestPoint:TestPoint_Pad_D1.5mm, F.Cu at (167.4, 249.5)
- added TP24: DMD_LAT, TestPoint:TestPoint_Pad_D1.5mm, F.Cu at (152.2, 253.9)
- added U27: 74AHCT245, Package_SO:TSSOP-20_4.4x6.5mm_P0.65mm, F.Cu at (156.4, 220.6)
- added U28: 74AHCT245, Package_SO:TSSOP-20_4.4x6.5mm_P0.65mm, F.Cu at (156.4, 231.5)
- added U29: 74AHCT245, Package_SO:TSSOP-20_4.4x6.5mm_P0.65mm, F.Cu at (156.4, 242.4)
- added U30: 74HC165, Package_SO:SOIC-16_3.9x9.9mm_P1.27mm, F.Cu at (52.2, 189.9)
- added U31: 74HC595, Package_SO:SOIC-16_3.9x9.9mm_P1.27mm, F.Cu at (139.3, 250.8)
Connections:
- J21 pad 16: Net-(J21-GPIO23) -> RP_IRQ_N
- J21 pad 19: Net-(J21-MOSI0/GPIO10) -> FRAME_MOSI
- J21 pad 23: Net-(J21-SCLK0/GPIO11) -> FRAME_SCK
- J21 pad 24: Net-(J21-~{CE0}/GPIO8) -> FRAME_CS_N
- R17 pad 2: Net-(U4-GPIO42/ADC2) -> LED_STATUS
- R176 pad 1: DMD_DE -> DMD_D0
- R177 pad 1: DMD_ROWDATA -> DMD_D1
- R178 pad 1: DMD_ROWCLK -> DMD_D2
- R179 pad 1: DMD_COLLATCH_A -> DMD_D3
- R18 pad 2: Net-(U4-GPIO33) -> RP_UART_RX
- R180 pad 1: DMD_PIXCLK -> DMD_D4
- R181 pad 1: DMD_SDATA -> DMD_D5
- R182 pad 1: DMD_COLLATCH_B -> DMD_D6
- R19 pad 2: Net-(U4-GPIO32) -> RP_UART_TX
- R22 pad 2: Net-(J21-GPIO23) -> RP_IRQ_N
- U19 pad 9: SW_DATA -> CHAIN6
- U20 pad 12: STB_LATCH -> SW_LOAD_N
- U20 pad 14: STB_DATA -> STB_CHAIN
- U21 pad 2: DMD_DE -> DMD_D0
- U21 pad 3: DMD_ROWDATA -> DMD_D1
- U21 pad 4: DMD_ROWCLK -> DMD_D2
- U21 pad 5: DMD_COLLATCH_A -> DMD_D3
- U21 pad 6: DMD_PIXCLK -> DMD_D4
- U21 pad 7: DMD_SDATA -> DMD_D5
- U21 pad 8: DMD_COLLATCH_B -> DMD_D6
- U4 pad 20: STB_LATCH -> DMD_D0
- U4 pad 21: DMD_DE -> DMD_D1
- U4 pad 22: DMD_ROWDATA -> DMD_D2
- U4 pad 23: DMD_ROWCLK -> DMD_D3
- U4 pad 25: DMD_COLLATCH_A -> DMD_D4
- U4 pad 26: DMD_PIXCLK -> DMD_D5
- U4 pad 27: DMD_SDATA -> DMD_D6
- U4 pad 28: DMD_COLLATCH_B -> DMD_D7
- U4 pad 36: Net-(J21-MOSI0/GPIO10) -> DMD_D8
- U4 pad 37: Net-(J21-~{CE0}/GPIO8) -> DMD_D9
- U4 pad 38: Net-(J21-SCLK0/GPIO11) -> DMD_D10
- U4 pad 39: MEM_PROTECT -> DMD_D11
- U4 pad 40: Net-(U4-GPIO32) -> DMD_CLK
- U4 pad 42: Net-(U4-GPIO33) -> DMD_LAT
- U4 pad 43: Net-(J21-GPIO23) -> DMD_OE
- U4 pad 44: GI_PWM -> DMD_A
- U4 pad 45: GI_SPARE -> DMD_B
- U4 pad 46: AMP_MUTE -> RP_IRQ_N
- U4 pad 47: unconnected-(U4-GPIO38-Pad47) -> GI_PWM
- U4 pad 48: unconnected-(U4-GPIO39-Pad48) -> AMP_MUTE
- U4 pad 49: VMON_5V -> FRAME_MOSI
- U4 pad 52: VMON_12V -> FRAME_CS_N
- U4 pad 53: Net-(U4-GPIO42/ADC2) -> FRAME_SCK
- U4 pad 55: unconnected-(U4-GPIO44/ADC4-Pad55) -> RP_UART_TX
- U4 pad 56: unconnected-(U4-GPIO45/ADC5-Pad56) -> RP_UART_RX
- U4 pad 57: unconnected-(U4-GPIO46/ADC6-Pad57) -> VMON_5V
- U4 pad 58: unconnected-(U4-GPIO47/ADC7-Pad58) -> VMON_12V
Other:
- board size 120.7 x 231.8 mm -> 142 x 231.8 mm
