File: hardware/kicad/sam_cpu/sam_cpu.kicad_pcb (KiCad board)
At the start: 4 copper layers, 142 x 236.8 mm, 459 parts, among them J1 J1 SWITCH COLUMNS, J10 J10 SPEAKERS, J11 J11 POWER, J12 J12 SWITCH ROWS, J13 J13 DEDICATED, J17 EXT 5V, J18 J18 GI DIMMER, J19 USB-C (to Pi), J2 J2 DEDICATED, J20 SWD, J21 Raspberry Pi 40-pin, J22 J22 STEREO, J23 EXT 12V, J24 J24 SUBWOOFER, J27 J27 RS485 IN, J28 J28 I2S IN, J29 J29 RS485 OUT, J3 J3 DEDICATED, J30 J30 LINE IN, J6 J6 SWITCH ROWS, J9 J9 IO BUS, Q1 AO3401A, Q11 MMBT3904, Q12 MMBT3904, Q13 MMBT3904, Q14 MMBT3904, Q15 MMBT3904, Q16 MMBT3904, Q17 MMBT3904, Q18 MMBT3904, Q2 AO3401A, Q3 2N7002, Q4 2N7002, SW1 RESET, SW2 BOOTSEL, SW3 DIP x8, U1 LTC4412, U10 LM339, U11 LM339, U14 74HC165, U15 74HC165, U16 74HC165, U17 74HC165, U18 74HC165, U19 74HC165, U2 LTC4412, U20 74HC595, U22 PCM5102A, U23 TDA7297, U24 TDA7297, U25 DS3231MZ, U26 OPA1678, U3 NCP1117-3.3, U30 74HC165, U31 74HC595, U32 ADM2682E, U4 RP2354B, U5 TPS3808G33, U6 SN74LVC8T245, U7 74AHCT541, U8 LM339, U9 LM339, Y1 12MHz

Commit message: Schematic: put the Pi header 3V3 pins on a PI_3V3 net instead of a no-connect
J21 pins 1 and 17 (the Pi's own 3V3 output) sat on a no-connect flag, so KiCad
named the pair unconnected-(J21-3V3-Pad1) and asked for the two pads to be
joined. They now carry a PI_3V3 label with a PWR_FLAG (the Pi drives it); ERC
is unchanged apart from the library-path warning every power symbol has.
The boards take the new net name on the same pads and tracks: the Freerouting
board and KRT run A already join the two pins, run C still needs the track.

Co-Authored-By: Claude Opus 5.5 (1M context) <noreply@anthropic.com>
Claude-Session: https://claude.ai/code/session_012mQXTyxPh1ZSDfsNXZEFhJ
Connections:
- J21 pad 1: unconnected-(J21-3V3-Pad1) -> /MCU and Pi/PI_3V3
- J21 pad 17: unconnected-(J21-3V3-Pad1) -> /MCU and Pi/PI_3V3
Routing:
- net unconnected-(J21-3V3-Pad1): track 24.8 -> 0.00 mm
- net /MCU and Pi/PI_3V3: track 0.00 -> 24.8 mm
Changed lines of the file:
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@@
 			(layers "*.Cu" "*.Mask")
 			(remove_unused_layers no)
-			(net "unconnected-(J21-3V3-Pad1)")
+			(net "/MCU and Pi/PI_3V3")
 		)
 		(pad "2" thru_hole circle
@@
 			(layers "*.Cu" "*.Mask")
 			(remove_unused_layers no)
-			(net "unconnected-(J21-3V3-Pad1)")
+			(net "/MCU and Pi/PI_3V3")
 		)
 		(pad "18" thru_hole circle
@@
 		(width 0.2)
 		(layer "B.Cu")
-		(net "unconnected-(J21-3V3-Pad1)")
+		(net "/MCU and Pi/PI_3V3")
 	)
 	(segment
@@
 		(width 0.2)
 		(layer "B.Cu")
-		(net "unconnected-(J21-3V3-Pad1)")
+		(net "/MCU and Pi/PI_3V3")
 	)
 	(segment
@@
 		(width 0.2)
 		(layer "B.Cu")
-		(net "unconnected-(J21-3V3-Pad1)")
+		(net "/MCU and Pi/PI_3V3")
 	)
 	(segment
@@
 		(width 0.2)
 		(layer "B.Cu")
-		(net "unconnected-(J21-3V3-Pad1)")
+		(net "/MCU and Pi/PI_3V3")
 	)
 	(segment
@@
 		(width 0.2)
 		(layer "B.Cu")
-		(net "unconnected-(J21-3V3-Pad1)")
+		(net "/MCU and Pi/PI_3V3")
 	)
 	(segment
@@
 		(width 0.2)
 		(layer "B.Cu")
-		(net "unconnected-(J21-3V3-Pad1)")
+		(net "/MCU and Pi/PI_3V3")
 	)
 	(segment
@@
 		(width 0.15)
 		(layer "B.Cu")
-		(net "unconnected-(J21-3V3-Pad1)")
+		(net "/MCU and Pi/PI_3V3")
 	)
 	(segment
@@
 		(width 0.2)
 		(layer "B.Cu")
-		(net "unconnected-(J21-3V3-Pad1)")
+		(net "/MCU and Pi/PI_3V3")
 	)
 	(segment
@@
 		(width 0.2)
 		(layer "B.Cu")
-		(net "unconnected-(J21-3V3-Pad1)")
+		(net "/MCU and Pi/PI_3V3")
 	)
 	(segment
@@
 		(width 0.2)
 		(layer "B.Cu")
-		(net "unconnected-(J21-3V3-Pad1)")
+		(net "/MCU and Pi/PI_3V3")
 	)
 	(segment
@@
 		(width 0.2)
 		(layer "B.Cu")
-		(net "unconnected-(J21-3V3-Pad1)")
+		(net "/MCU and Pi/PI_3V3")
 	)
 	(segment
@@
 		(width 0.2)
 		(layer "B.Cu")
-		(net "unconnected-(J21-3V3-Pad1)")
+		(net "/MCU and Pi/PI_3V3")
 	)
 	(segment
@@
 		(width 0.2)
 		(layer "B.Cu")
-		(net "unconnected-(J21-3V3-Pad1)")
+		(net "/MCU and Pi/PI_3V3")
 	)
 	(segment
@@
 		(width 0.15)
 		(layer "B.Cu")
-		(net "unconnected-(J21-3V3-Pad1)")
+		(net "/MCU and Pi/PI_3V3")
 	)
 	(segment
