File: hardware/kicad/sam_cpu/mcu.kicad_sch (KiCad schematic)
At the start: 50 parts, among them J19 USB-C (to Pi), J20 SWD, J21 Raspberry Pi 40-pin, SW1 RESET, SW2 BOOTSEL, U25 DS3231MZ, U4 RP2354B, U5 TPS3808G33, Y1 12MHz

Commit message: Schematic: put the Pi header 3V3 pins on a PI_3V3 net instead of a no-connect
J21 pins 1 and 17 (the Pi's own 3V3 output) sat on a no-connect flag, so KiCad
named the pair unconnected-(J21-3V3-Pad1) and asked for the two pads to be
joined. They now carry a PI_3V3 label with a PWR_FLAG (the Pi drives it); ERC
is unchanged apart from the library-path warning every power symbol has.
The boards take the new net name on the same pads and tracks: the Freerouting
board and KRT run A already join the two pins, run C still needs the track.

Co-Authored-By: Claude Opus 5.5 (1M context) <noreply@anthropic.com>
Claude-Session: https://claude.ai/code/session_012mQXTyxPh1ZSDfsNXZEFhJ
Connections:
- net PI_3V3: now reaches J21.1 (3V3), J21.17 (3V3)
- no-connect marks 37 -> 36
Changed lines of the file:
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@@
 		(at 40.64 147.32)
 	)
-	(no_connect
-		(at 320.04 134.62)
+	(wire
+		(pts
+			(xy 320.04 134.62) (xy 320.04 132.08)
+		)
+		(stroke
+			(width 0)
+			(type default)
+		)
+	)
+	(wire
+		(pts
+			(xy 320.04 132.08) (xy 320.04 129.54)
+		)
+		(stroke
+			(width 0)
+			(type default)
+		)
+	)
+	(label "PI_3V3"
+		(at 320.04 129.54 90)
+		(effects
+			(font
+				(size 1.27 1.27)
+			)
+			(justify left bottom)
+		)
+	)
+	(symbol
+		(lib_id "power:PWR_FLAG")
+		(at 320.04 132.08 90)
+		(unit 1)
+		(body_style 1)
+		(exclude_from_sim no)
+		(in_bom no)
+		(on_board no)
+		(in_pos_files yes)
+		(dnp no)
+		(property "Reference" "#FLG1303"
+			(at 316.23 132.08 0)
+			(hide yes)
+			(show_name no)
+			(do_not_autoplace no)
+			(effects
+				(font
+					(size 1.27 1.27)
+				)
+			)
+		)
+		(property "Value" "PWR_FLAG"
+			(at 314.96 132.08 0)
+			(show_name no)
+			(do_not_autoplace no)
+			(effects
+				(font
+					(size 1.27 1.27)
+				)
+			)
+		)
+		(property "Footprint" ""
+			(at 320.04 132.08 0)
+			(hide yes)
+			(show_name no)
+			(do_not_autoplace no)
+			(effects
+				(font
+					(size 1.27 1.27)
+				)
+			)
+		)
+		(property "Datasheet" ""
+			(at 320.04 132.08 0)
+			(hide yes)
+			(show_name no)
+			(do_not_autoplace no)
+			(effects
+				(font
+					(size 1.27 1.27)
+				)
+			)
+		)
+		(property "Description" "Special symbol for telling ERC where power comes from"
+			(at 320.04 132.08 0)
+			(hide yes)
+			(show_name no)
+			(do_not_autoplace no)
+			(effects
+				(font
+					(size 1.27 1.27)
+				)
+			)
+		)
+		(pin "1"
+		)
+		(instances
+			(project "sam_cpu"
+				(path "/2aea4fdf-a573-57d0-a5af-7bd6ce737647/d360c6c3-40d3-5528-aec0-e616a30a2847"
+					(reference "#FLG1303")
+					(unit 1)
+				)
+			)
+		)
 	)
 	(no_connect
