File: hardware/kicad/sam_cpu/mcu.kicad_sch (KiCad schematic)
At the start: 50 parts, among them J19 USB-C (to Pi), J20 SWD, J21 Raspberry Pi 40-pin, SW1 RESET, SW2 BOOTSEL, U25 DS3231MZ, U4 RP2354B, U5 TPS3808G33, Y1 12MHz

Commit message: U32 CA-IS2092VW, BT1 XDCR-2032, J27/J29 side-entry RJ45 for JLCPCB stock
Replace parts JLCPCB does not stock: U32 ADM2682E -> CA-IS2092VW (new symbol,
pinout remap), BT1 Keystone 3034 -> Lianxin XDCR-2032-603, J27/J29 OST PJ012 ->
CONNFLY DS1128-05-S8B8P side-entry at the right edge. Isolated side and BT1
rerouted; project footprint library sam_cpu.pretty added.

Co-Authored-By: Claude Opus 5.5 (1M context) <noreply@anthropic.com>
Claude-Session: https://claude.ai/code/session_01ExuDVoDDDHhVWjb8EwVzYb
Parts:
- BT1: footprint Battery:BatteryHolder_Keystone_3034_1x20mm -> sam_cpu:BatteryHolder_Lianxin_XDCR-2032-603
Changed lines of the file:
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@@
 			)
 		)
-		(property "Footprint" "Battery:BatteryHolder_Keystone_3034_1x20mm"
+		(property "Footprint" "sam_cpu:BatteryHolder_Lianxin_XDCR-2032-603"
 			(at 45.72 257.556 90)
 			(hide yes)

Commit message: J19/J30 to JLCPCB-stocked parts (SH-U262-161N-4BVC11, PJ-393-7A)
J19 keeps the TYPE-C-31-M-12 pattern with the clone's longer rear shell slots.
J30 becomes the SMD PJ-393-7A switched stereo jack from the maker's drawing;
+12V, I2S_DIN, FRAME_SCK and the audio nets are rerouted around its pads.
Both footprints are added to sam_cpu.pretty. DRC and parity unchanged.

Co-Authored-By: Claude Opus 5.5 (1M context) <noreply@anthropic.com>
Claude-Session: https://claude.ai/code/session_01ExuDVoDDDHhVWjb8EwVzYb
Parts:
- J19: footprint Connector_USB:USB_C_Receptacle_HRO_TYPE-C-31-M-12 -> sam_cpu:USB_C_Receptacle_SH_U262-161N-4BVC11
Changed lines of the file:
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@@
 			)
 		)
-		(property "Footprint" "Connector_USB:USB_C_Receptacle_HRO_TYPE-C-31-M-12"
+		(property "Footprint" "sam_cpu:USB_C_Receptacle_SH_U262-161N-4BVC11"
 			(at 29.21 132.08 0)
 			(hide yes)

Commit message: Remove USB-C, GI dimmer, SWD header and DIP block; Pi SWD on GPIO24/25 as raspberrypi-swd.cfg
c35 (schematic) and c36 (board): J19 with R10-R14, the GI dimmer sheet (J18, R183-R185),
J20, and the DIP block (SW3, R168-R175, C93, U14) go to free routing space. U15's serial
input goes to GND. J21 pin 18 (GPIO24) is now SWDIO and pin 22 (GPIO25) SWCLK, matching
Raspberry Pi's OpenOCD interface/raspberrypi-swd.cfg. ERC clean, schematic parity clean.

Co-Authored-By: Claude Opus 5.5 (1M context) <noreply@anthropic.com>
Claude-Session: https://claude.ai/code/session_01QQate2kninVTv93dgZ4pfZ
Parts:
- removed J19: USB-C (to Pi), sam_cpu:USB_C_Receptacle_SH_U262-161N-4BVC11, symbol Connector:USB_C_Receptacle_USB2.0_16P
- removed J20: SWD, Connector_PinHeader_2.54mm:PinHeader_1x03_P2.54mm_Vertical, symbol Connector_Generic:Conn_01x03
- removed R10: 100k, Resistor_SMD:R_0603_1608Metric, symbol Device:R
- removed R11, R12: 5.1k, Resistor_SMD:R_0603_1608Metric, symbol Device:R
- removed R13, R14: 27, Resistor_SMD:R_0603_1608Metric, symbol Device:R
Connections:
- net SWCLK: now also J21.22 (GPIO25); no longer J21.18 (GPIO24)
- net SWDIO: now also J21.18 (GPIO24); no longer J21.22 (GPIO25)
- net GI_PWM: no longer names the net of U4.47 (GPIO38)
- no-connect marks 36 -> 37
Other:
- note added: "GPIO map: ARCHITECTURE.md 9.2. PIO0 bus on GPIO0-15, PIO1 switch chain on GPIO16-20, GPIO20-22: RS485 port (UART1 TX / RX, driver enable, page 13); GPIO23-36 unassigned. Pi UART3 (GPIO4 / 5, RTS on GPIO7) reaches the same port. Frames from the Pi on SPI1 (GPIO40-42), UART0 on GPIO44-45, ADC monitors on GPIO46-47, GPIO43 spare. Coin door and status LED moved onto the switch chain. No USB: the Pi f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"
- note removed: "GPIO map: ARCHITECTURE.md 9.2. PIO0 bus on GPIO0-15, PIO1 switch chain on GPIO16-20, GPIO20-22: RS485 port (UART1 TX / RX, driver enable, page 13); GPIO23-36 unassigned. Pi UART3 (GPIO4 / 5, RTS on GPIO7) reaches the same port. Frames from the Pi on SPI1 (GPIO40-42), UART0 on GPIO44-45, ADC monitors on GPIO46-47, GPIO43 spare. Coin door, status LED and GI_SPARE moved onto the switch chain. Core s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"

Commit message: Put USB-C J19 back (placed, unrouted) with a USB differential pair class
c38 (schematic): J19 and R10-R14 return on the MCU sheet as at e6c37a8; the
pair is named USB_D+ / USB_D- (U4 to R13 / R14) and USB_C_D+ / USB_C_D- (to
J19). c39 (board): J19 / R13 / R14 at their old spots above U4, R10-R12 in a
column left of J19, 1 mm or more between courtyards, no routing. Netclass USB
(0.2 mm / 0.15 mm gap pair) and a DRC rule for gap, uncoupled length and skew.
J20, the GI dimmer and the DIP block stay removed. 28 unconnected items (18 +
10 for USB-C), ERC clean, no new DRC errors.

Co-Authored-By: Claude Opus 5.5 (1M context) <noreply@anthropic.com>
Claude-Session: https://claude.ai/code/session_01QQate2kninVTv93dgZ4pfZ
Parts:
- added J19: USB-C (to Pi), sam_cpu:USB_C_Receptacle_SH_U262-161N-4BVC11, symbol Connector:USB_C_Receptacle_USB2.0_16P
- added R10: 100k, Resistor_SMD:R_0603_1608Metric, symbol Device:R
- added R11, R12: 5.1k, Resistor_SMD:R_0603_1608Metric, symbol Device:R
- added R13, R14: 27, Resistor_SMD:R_0603_1608Metric, symbol Device:R
Connections:
- net GND: now also J19.A1 (GND), J19.A12 (GND), J19.B1 (GND), J19.B12 (GND), J19.SH (SHIELD), R10.2, R11.2, R12.2
- net USB_D-: now reaches U4.66 (USB_DM)
- net USB_D-: now also R13.2
- net USB_D+: now reaches U4.67 (USB_DP)
- net USB_D+: now also R14.2
- new net: J19.A4 (VBUS), J19.A9 (VBUS), J19.B4 (VBUS), J19.B9 (VBUS), R10.1
- new net: J19.B5 (CC2), R12.1
- new net: J19.A5 (CC1), R11.1
- new net USB_C_D+: J19.A6 (D+), J19.B6 (D+), R14.1
- new net USB_C_D-: J19.A7 (D-), J19.B7 (D-), R13.1
Other:
- note added: "GPIO map: ARCHITECTURE.md 9.2. PIO0 bus on GPIO0-15, PIO1 switch chain on GPIO16-20, GPIO20-22: RS485 port (UART1 TX / RX, driver enable, page 13); GPIO23-36 unassigned. Pi UART3 (GPIO4 / 5, RTS on GPIO7) reaches the same port. Frames from the Pi on SPI1 (GPIO40-42), UART0 on GPIO44-45, ADC monitors on GPIO46-47, GPIO43 spare. Coin door and status LED moved onto the switch chain. USB-C J19 (backu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"
- note removed: "GPIO map: ARCHITECTURE.md 9.2. PIO0 bus on GPIO0-15, PIO1 switch chain on GPIO16-20, GPIO20-22: RS485 port (UART1 TX / RX, driver enable, page 13); GPIO23-36 unassigned. Pi UART3 (GPIO4 / 5, RTS on GPIO7) reaches the same port. Frames from the Pi on SPI1 (GPIO40-42), UART0 on GPIO44-45, ADC monitors on GPIO46-47, GPIO43 spare. Coin door and status LED moved onto the switch chain. No USB: the Pi f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"

Commit message: Clean +12 V rail (ideal-diode OR of J23 and J11 pin 6) and a Pi buck with BUCK / BOARD jumpers
c42 (schematic): LTC4412 + DMP3013SFV per input into F1, external priority via
the U34 CTL divider; TPS54302 buck to PI_5V_BUCK; JP4 BUCK / JP3 BOARD pick the
J21 5 V (both open for a Jetson). c43 (board): OR by J23, buck under the Pi,
JP3 cuts the +5V trunk to J21, all hand-routed; 23 unconnected as before, no
new DRC errors.

Co-Authored-By: Claude Opus 5.5 <noreply@anthropic.com>
Claude-Session: https://claude.ai/code/session_01QQate2kninVTv93dgZ4pfZ
Connections:
- net +5V renamed PI_5V
Changed lines of the file:
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@@
 	)
 	(symbol
-		(lib_id "power:+5V")
-		(at 330.2 132.08 0)
-		(unit 1)
-		(body_style 1)
-		(exclude_from_sim no)
-		(in_bom no)
-		(on_board no)
-		(in_pos_files yes)
-		(dnp no)
-		(property "Reference" "#PWR02056"
-			(at 330.2 135.89 0)
-			(hide yes)
-			(show_name no)
-			(do_not_autoplace no)
-			(effects
-				(font
-					(size 1.6 1.6)
-				)
-			)
-		)
-		(property "Value" "+5V"
-			(at 330.2 128.524 0)
-			(show_name no)
-			(do_not_autoplace no)
-			(effects
-				(font
-					(size 1.6 1.6)
-				)
-			)
-		)
-		(property "Footprint" ""
-			(at 330.2 132.08 0)
-			(hide yes)
-			(show_name no)
-			(do_not_autoplace no)
-			(effects
-				(font
-					(size 1.6 1.6)
-				)
-			)
-		)
-		(property "Datasheet" ""
-			(at 330.2 132.08 0)
-			(hide yes)
-			(show_name no)
-			(do_not_autoplace no)
-			(effects
-				(font
-					(size 1.6 1.6)
-				)
-			)
-		)
-		(property "Description" "Power symbol creates a global label with name \"+5V\""
-			(at 330.2 132.08 0)
-			(hide yes)
-			(show_name no)
-			(do_not_autoplace no)
-			(effects
-				(font
-					(size 1.6 1.6)
-				)
-			)
-		)
-		(pin "1"
-		)
-		(instances
-			(project "sam_cpu"
-				(path "/2aea4fdf-a573-57d0-a5af-7bd6ce737647/d360c6c3-40d3-5528-aec0-e616a30a2847"
-					(reference "#PWR02056")
-					(unit 1)
-				)
-			)
-		)
-	)
-	(symbol
 		(lib_id "power:+1V1")
 		(at 203.2 63.5 0)
@@
 		)
 	)
+	(global_label "PI_5V"
+		(shape passive)
+		(at 330.2 132.08 90)
+		(fields_autoplaced yes)
+		(effects
+			(font
+				(size 1.6 1.6)
+			)
+			(justify left)
+		)
+		(property "Intersheetrefs" "${INTERSHEET_REFS}"
+			(at 330.2 132.08 0)
+			(hide yes)
+			(show_name no)
+			(do_not_autoplace no)
+			(effects
+				(font
+					(size 1.6 1.6)
+				)
+				(justify left)
+			)
+		)
+	)
