File: hardware/kicad/sam_cpu/sam_cpu.kicad_sch (KiCad schematic)
At the start: 0 parts

Commit message: Remove USB-C, GI dimmer, SWD header and DIP block; Pi SWD on GPIO24/25 as raspberrypi-swd.cfg
c35 (schematic) and c36 (board): J19 with R10-R14, the GI dimmer sheet (J18, R183-R185),
J20, and the DIP block (SW3, R168-R175, C93, U14) go to free routing space. U15's serial
input goes to GND. J21 pin 18 (GPIO24) is now SWDIO and pin 22 (GPIO25) SWCLK, matching
Raspberry Pi's OpenOCD interface/raspberrypi-swd.cfg. ERC clean, schematic parity clean.

Co-Authored-By: Claude Opus 5.5 (1M context) <noreply@anthropic.com>
Claude-Session: https://claude.ai/code/session_01QQate2kninVTv93dgZ4pfZ
Other:
- removed sheet GI dimmer
- note added: "Dedicated switches D17-D24 (J13)"
- note removed: "Dedicated switches D17-D24 (J13) and DIP switches"
- note removed: "J18 GI dimmer header"
Changed lines of the file:
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@@
 		(company "Stern SAM CPU PPUC (CERN-OHL-S v2)")
 	)
-	(text "Dedicated switches D17-D24 (J13) and DIP switches"
+	(text "Dedicated switches D17-D24 (J13)"
 		(exclude_from_sim no)
 		(at 154.94 160.02 0)
@@
 		(exclude_from_sim no)
 		(at 27.94 160.02 0)
-		(effects
-			(font
-				(size 1.6 1.6)
-			)
-			(justify left top)
-		)
-	)
-	(text "J18 GI dimmer header"
-		(exclude_from_sim no)
-		(at 281.94 160.02 0)
 		(effects
 			(font
@@
 				)
 			)
-		)
-	)
-	(sheet
-		(at 279.4 154.94)
-		(size 88.9 25.4)
-		(exclude_from_sim no)
-		(in_bom yes)
-		(on_board yes)
-		(dnp no)
-		(fields_autoplaced yes)
-		(stroke
-			(width 0.1524)
-			(type solid)
-		)
-		(fill
-			(color 0 0 0 0)
-		)
-		(property "Sheetname" "GI dimmer"
-			(at 279.4 154.2284 0)
-			(show_name no)
-			(do_not_autoplace no)
-			(effects
-				(font
-					(size 2 2)
-				)
-				(justify left bottom)
-			)
-		)
-		(property "Sheetfile" "display_gi.kicad_sch"
-			(at 279.4 180.9284 0)
-			(show_name no)
-			(do_not_autoplace no)
-			(effects
-				(font
-					(size 1.6 1.6)
-				)
-				(justify left top)
-			)
-		)
-		(instances
-			(project "sam_cpu"
-				(path "/2aea4fdf-a573-57d0-a5af-7bd6ce737647"
-					(page "10")
-				)
-			)
