File: hardware/sam_io_board/sam_io_krt/sam_io.kicad_pcb (KiCad board)
At the start: 2 copper layers, 100 x 70 mm, 104 parts, among them J1 Conn_01x06, J2 nmount JST 1mm QWIIC, J3 nmount SW Debug, J4 USB_C_Receptacle_USB2.0, J5 Conn_01x06, J9 SAM BUS, Q1 2N7002, SW1 Reset, SW2 Boot, SW3 ADDRESS, U1 ADM3483, U2 W25Q128JVSIQ, U3 RP2040, U4 LMV321, U5 SN74AHCT1G125, U6 AP2112K-3.3, U7 SN74LVC8T245, U8 74AHCT541, Y1 12MHz,18pF

Commit message: SAM_IO: remove the QWIIC option (J2, R96, R97, C8); R9 becomes a track
Schematic: J2 and its pull-ups and decoupling removed, the 0 ohm R9 (U1 RO to GPIO1) replaced by a wire.
../sam_io board: the parts and their stubs removed. R9 cannot be a straight track because /485_DE runs
between its pads, so RO hops through one via on B.Cu to the existing /485_RX via. DRC: 0 unconnected,
0 clearance, schematic parity clean apart from the existing field differences.
sam_io_krt (0.15 mm) board: same removal, R9 as a straight F.Cu track, DRC unchanged.

Co-Authored-By: Claude Opus 5.5 (1M context) <noreply@anthropic.com>
Claude-Session: https://claude.ai/code/session_012ePkTGNjii74e9emvMVPmF
Parts:
- removed C8: 100n, Capacitor_SMD:C_0402_1005Metric
- removed J2: nmount JST 1mm QWIIC, Connector_JST:JST_SH_SM04B-SRSS-TB_1x04-1MP_P1.00mm_Horizontal
- removed R9: 0, Resistor_SMD:R_0603_1608Metric
- removed R96, R97: 10k, Resistor_SMD:R_0603_1608Metric
Connections:
- U1 pad 1: Net-(U1-RO) -> /485_RX
Routing:
- net /485_TX: track 59.7 -> 21.3 mm, vias 8 -> 4
- net /485_RX: track 55.5 -> 28.3 mm, vias 6 -> 4
- net +3V3: track 222.3 -> 217.5 mm
- net Net-(U1-RO): track 3.57 -> 0.00 mm
