File: hardware/sam_io_board/sam_io_krt/escape/sam_io.kicad_pcb (KiCad board)
At the start: 2 copper layers, 100 x 70 mm, 104 parts, among them J1 Conn_01x06, J2 nmount JST 1mm QWIIC, J3 nmount SW Debug, J4 USB_C_Receptacle_USB2.0, J5 Conn_01x06, J9 SAM BUS, Q1 2N7002, SW1 Reset, SW2 Boot, SW3 ADDRESS, U1 ADM3483, U2 W25Q128JVSIQ, U3 RP2040, U4 LMV321, U5 SN74AHCT1G125, U6 AP2112K-3.3, U7 SN74LVC8T245, U8 74AHCT541, Y1 12MHz,18pF

Commit message: sam_io_krt/escape: rerouted after the QWIIC removal, RS485 lines kept from ../sam_io
2 unconnected (/nReset, GPIO25), 0 clearance at the board's own 0.2 mm rules.

Co-Authored-By: Claude Opus 5.5 (1M context) <noreply@anthropic.com>
Claude-Session: https://claude.ai/code/session_012ePkTGNjii74e9emvMVPmF
Parts:
- removed C8: 100n, Capacitor_SMD:C_0402_1005Metric
- removed J2: nmount JST 1mm QWIIC, Connector_JST:JST_SH_SM04B-SRSS-TB_1x04-1MP_P1.00mm_Horizontal
- removed R9: 0, Resistor_SMD:R_0603_1608Metric
- removed R96, R97: 10k, Resistor_SMD:R_0603_1608Metric
Connections:
- U1 pad 1: Net-(U1-RO) -> /485_RX
Routing:
- net GND: track 620.1 -> 286.4 mm, vias 33 -> 21
- net /485_TX: track 63.4 -> 26.1 mm, vias 5 -> 0
- net +3V3: track 219.5 -> 199.7 mm, vias 21 -> 22
- net Net-(J9-Pin_7): track 75.9 -> 92.9 mm, vias 2 -> 5
- net +5V: track 123.4 -> 134.4 mm
- net /B: track 48.6 -> 58.0 mm, vias 2 -> 1
- net /485_DE: track 25.0 -> 34.0 mm, vias 4 -> 0
- net Net-(J9-Pin_12): track 43.0 -> 37.4 mm, vias 2 -> 0
- net /485_RX: track 51.6 -> 47.1 mm
- net Net-(U1-RO): track 3.57 -> 0.00 mm
- net Net-(J9-Pin_5): track 26.5 -> 29.3 mm
- net Net-(J9-Pin_13): track 53.5 -> 51.5 mm, vias 0 -> 1
- net /nReset: track 9.93 -> 8.90 mm
- net Net-(J9-Pin_4): track 7.40 -> 8.11 mm
- net /A: track 44.6 -> 44.0 mm, vias 2 -> 3
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