File: hardware/sam_io_board/sam_io_100mm/sam_io.kicad_pcb (KiCad board)
At the start: 2 copper layers, 100 x 100 mm, 162 parts, among them J1 Conn_01x06, J13 J13 DEDICATED D17-D24, J2 J2 DEDICATED D1-D8, J20 nmount SW Debug, J3 J3 DEDICATED D9-D16, J4 USB_C_Receptacle_USB2.0, J5 Conn_01x06, J9 SAM BUS, Q1 2N7002, SW1 Reset, SW2 Boot, SW3 ADDRESS, U1 ADM3483, U3 RP2354B, U4 LMV321, U5 SN74AHCT1G125, U6 AP2112K-3.3, U7 SN74LVC8T245, U8 74AHCT541, Y1 12MHz,18pF

Commit message: SAM_IO 100 mm: move J3 3.5 mm down toward the bottom edge
Opens the gap between J2 and J3. IN_D9..IN_D16 rerouted (Freerouting plus
one A* route), one GND stitch via added; DRC 0 unconnected, only the known
J4 hole-clearance errors. J3 reference moved inside the board.

Co-Authored-By: Claude Opus 5.5 (1M context) <noreply@anthropic.com>
Claude-Session: https://claude.ai/code/session_01Mh8jyzQSZ4SYbwGJXqcn3P
Parts:
- moved J3 3.50 mm to (160.1, 132.5)
Routing:
- net /Dedicated switches/IN_D12: track 144.2 -> 94.0 mm, vias 3 -> 2
- net /Dedicated switches/IN_D10: track 136.5 -> 157.9 mm, vias 2 -> 3
- net /Dedicated switches/IN_D13: track 102.3 -> 88.6 mm, vias 3 -> 2
- net /Dedicated switches/IN_D11: track 112.7 -> 118.8 mm, vias 6 -> 4
- net /Dedicated switches/IN_D16: track 64.9 -> 70.9 mm, vias 2 -> 1
- net /Dedicated switches/IN_D9: track 159.9 -> 154.3 mm, vias 3 -> 1
- net /Dedicated switches/IN_D15: track 76.3 -> 80.6 mm
- net /Dedicated switches/IN_D14: track 93.1 -> 91.4 mm, vias 3 -> 1
- net DED_D23: track 58.7 -> 59.4 mm
- net GND: vias 281 -> 282

Commit message: SAM_IO rev 0.2: move J9 to the left edge, turned like the CPU board's J9
J9 now stands vertical on the left edge above J13 on both boards: pin 1 at
the bottom, odd pins and the key notch toward the board centre, as on the
SAM CPU board, so the IO board ribbon arrives from the same side. Bus nets
rerouted with Freerouting (other tracks locked); on the 100 mm board the
logo moved to the old J9 spot, one GND stitch via added and two isolated
stitch vias removed. DRC 0 unconnected on both boards.

Co-Authored-By: Claude Opus 5.5 (1M context) <noreply@anthropic.com>
Claude-Session: https://claude.ai/code/session_01Mh8jyzQSZ4SYbwGJXqcn3P
Parts:
- moved J9 60.2 mm to (91.5, 70.0), turned to 180 degrees
Routing:
- net Net-(J9-Pin_1): track 7.64 -> 89.1 mm, vias 0 -> 1
- net Net-(J9-Pin_6): track 5.19 -> 76.4 mm, vias 1 -> 2
- net Net-(J9-Pin_5): track 8.00 -> 79.2 mm, vias 0 -> 1
- net Net-(J9-Pin_8): track 5.31 -> 67.2 mm
- net Net-(J9-Pin_3): track 8.00 -> 65.8 mm
- net Net-(J9-Pin_4): track 8.23 -> 64.0 mm
- net Net-(J9-Pin_2): track 11.7 -> 63.6 mm, vias 1 -> 2
- net Net-(J9-Pin_16): track 4.90 -> 46.2 mm, vias 0 -> 2
- net Net-(J9-Pin_18): track 6.68 -> 46.8 mm, vias 1 -> 2
- net Net-(J9-Pin_14): track 9.97 -> 45.0 mm, vias 0 -> 1
- net Net-(J9-Pin_7): track 42.8 -> 60.2 mm, vias 1 -> 5
- net Net-(J9-Pin_15): track 25.4 -> 36.7 mm, vias 0 -> 1
- net Net-(J9-Pin_12): track 40.5 -> 48.3 mm, vias 1 -> 3
- net /Dedicated switches/IN_D15: track 80.6 -> 83.6 mm
- net Net-(J9-Pin_13): track 40.4 -> 38.8 mm
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